Commit message: Add config file for proto2

File: r2p_sea_arm_description/urdf/r2p_sea_arm_right.xacro (robot description, xacro)
@@ -41,5 +41,5 @@
     <parent link="right_arm_link"/>
     <child link="right_shoulder_pitch_link"/>
-    <origin xyz="0 -0.0872 0.0762" rpy="0 0 0"/>
+    <origin xyz="0 -0.0872 0.0762" rpy="0 -0.2 0"/>
     <axis xyz="0 1 0"/>
     <dynamics damping="${damp}"/>

Commit message: Global Industrie demo last modifications

File: r2p_sea_arm_description/urdf/r2p_sea_arm_right.xacro (robot description, xacro)
@@ -41,5 +41,5 @@
     <parent link="right_arm_link"/>
     <child link="right_shoulder_pitch_link"/>
-    <origin xyz="0 -0.0872 0.0762" rpy="0 -0.2 0"/>
+    <origin xyz="0 -0.0872 0.0762" rpy="0 -0.06 0"/>
     <axis xyz="0 1 0"/>
     <dynamics damping="${damp}"/>
